File: Hardware/Ampelope.kicad_sch (KiCad schematic)
At the start: 14 parts, among them J1 B_In, J3 Eurorack_10_pin_power, J4 RM_OUT, U1 TL074

Commit message: Starting modelling attack curves from Roland clone ADSR
Parts:
- added Q?: 2N3904, Package_TO_SOT_THT:TO-92_Inline, symbol Transistor_BJT:2N3904
- added R? (x2): 1k, symbol Device:R_Small
- J1: value B_In -> Gate1_In
Connections:
- net +3V3: now also R?.2
- net GND: now also Q?.1 (E)
- net Gate1_Inv: now reaches U?.40 (PC8)
- net Gate1_Inv: now also Q?.3 (C), R?.1
- net B_Input: no longer names the net of J1.3
- net B_Input: now also R?.1
- new net: Q?.2 (B), R?.2
Other:
- moved on the sheet: J1
Changed lines of the file:
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@@
   (junction (at 146.05 177.8) (diameter 1.016) (color 0 0 0 0))
   (junction (at 158.75 167.64) (diameter 1.016) (color 0 0 0 0))
-  (no_connect (at 217.17 60.96))
+  (junction (at 166.37 36.83) (diameter 1.016) (color 0 0 0 0))
+  (no_connect (at 147.32 40.64))
   (no_connect (at 217.17 97.79))
   (wire (pts (xy 24.13 167.64) (xy 27.94 167.64))
@@
     (stroke (width 0) (type solid) (color 0 0 0 0))
   )
+  (wire (pts (xy 41.91 101.6) (xy 45.72 101.6))
+    (stroke (width 0) (type solid) (color 0 0 0 0))
+  )
   (wire (pts (xy 41.91 182.88) (xy 27.94 182.88))
     (stroke (width 0) (type solid) (color 0 0 0 0))
@@
     (stroke (width 0) (type solid) (color 0 0 0 0))
   )
+  (wire (pts (xy 147.32 43.18) (xy 152.4 43.18))
+    (stroke (width 0) (type solid) (color 0 0 0 0))
+  )
+  (wire (pts (xy 147.32 45.72) (xy 147.32 49.53))
+    (stroke (width 0) (type solid) (color 0 0 0 0))
+  )
   (wire (pts (xy 153.67 167.64) (xy 158.75 167.64))
     (stroke (width 0) (type solid) (color 0 0 0 0))
   )
+  (wire (pts (xy 157.48 43.18) (xy 158.75 43.18))
+    (stroke (width 0) (type solid) (color 0 0 0 0))
+  )
   (wire (pts (xy 158.75 167.64) (xy 158.75 163.83))
     (stroke (width 0) (type solid) (color 0 0 0 0))
@@
     (stroke (width 0) (type solid) (color 0 0 0 0))
   )
+  (wire (pts (xy 166.37 27.94) (xy 166.37 29.21))
+    (stroke (width 0) (type solid) (color 0 0 0 0))
+  )
+  (wire (pts (xy 166.37 34.29) (xy 166.37 36.83))
+    (stroke (width 0) (type solid) (color 0 0 0 0))
+  )
+  (wire (pts (xy 166.37 36.83) (xy 166.37 38.1))
+    (stroke (width 0) (type solid) (color 0 0 0 0))
+  )
+  (wire (pts (xy 166.37 36.83) (xy 181.61 36.83))
+    (stroke (width 0) (type solid) (color 0 0 0 0))
+  )
+  (wire (pts (xy 166.37 48.26) (xy 166.37 50.8))
+    (stroke (width 0) (type solid) (color 0 0 0 0))
+  )
   (wire (pts (xy 168.91 167.64) (xy 172.72 167.64))
     (stroke (width 0) (type solid) (color 0 0 0 0))
@@
   )
   (wire (pts (xy 214.63 92.71) (xy 214.63 100.33))
-    (stroke (width 0) (type solid) (color 0 0 0 0))
-  )
-  (wire (pts (xy 217.17 63.5) (xy 227.33 63.5))
-    (stroke (width 0) (type solid) (color 0 0 0 0))
-  )
-  (wire (pts (xy 217.17 66.04) (xy 217.17 69.85))
     (stroke (width 0) (type solid) (color 0 0 0 0))
   )
@@
     (effects (font (size 1.27 1.27)) (justify right bottom))
   )
+  (label "Gate1_Inv" (at 41.91 101.6 180)
+    (effects (font (size 1.27 1.27)) (justify right bottom))
+  )
   (label "DAC3_1" (at 85.09 45.72 0)
     (effects (font (size 1.27 1.27)) (justify left bottom))
@@
     (effects (font (size 1.27 1.27)) (justify left bottom))
   )
-  (label "B_Input" (at 227.33 63.5 180)
+  (label "Gate1_Inv" (at 181.61 36.83 180)
     (effects (font (size 1.27 1.27)) (justify right bottom))
   )
@@
     (pin "1")
   )
+  (symbol (lib_id "power:+3.3V") (at 166.37 27.94 0) (unit 1)
+    (in_bom yes) (on_board yes) (fields_autoplaced)
+    (property "Reference" "#PWR?" (id 0) (at 166.37 31.75 0)
+      (effects (font (size 1.27 1.27)) hide)
+    )
+    (property "Value" "+3.3V" (id 1) (at 166.37 24.13 0))
+    (property "Footprint" "" (id 2) (at 166.37 27.94 0)
+      (effects (font (size 1.27 1.27)) hide)
+    )
+    (property "Datasheet" "" (id 3) (at 166.37 27.94 0)
+      (effects (font (size 1.27 1.27)) hide)
+    )
+    (pin "1")
+  )
   (symbol (lib_id "power:+3.3VA") (at 172.72 163.83 0) (unit 1)
     (in_bom yes) (on_board yes) (fields_autoplaced)
@@
     (pin "1")
   )
+  (symbol (lib_id "power:GND") (at 147.32 49.53 0) (unit 1)
+    (in_bom yes) (on_board yes) (fields_autoplaced)
+    (property "Reference" "#PWR08" (id 0) (at 147.32 55.88 0)
+      (effects (font (size 1.27 1.27)) hide)
+    )
+    (property "Value" "GND" (id 1) (at 147.32 54.61 0))
+    (property "Footprint" "" (id 2) (at 147.32 49.53 0)
+      (effects (font (size 1.27 1.27)) hide)
+    )
+    (property "Datasheet" "" (id 3) (at 147.32 49.53 0)
+      (effects (font (size 1.27 1.27)) hide)
+    )
+    (pin "1")
+  )
+  (symbol (lib_id "power:GND") (at 166.37 50.8 0) (unit 1)
+    (in_bom yes) (on_board yes)
+    (property "Reference" "#PWR?" (id 0) (at 166.37 57.15 0)
+      (effects (font (size 1.27 1.27)) hide)
+    )
+    (property "Value" "GND" (id 1) (at 166.497 55.1942 0))
+    (property "Footprint" "" (id 2) (at 166.37 50.8 0)
+      (effects (font (size 1.27 1.27)) hide)
+    )
+    (property "Datasheet" "" (id 3) (at 166.37 50.8 0)
+      (effects (font (size 1.27 1.27)) hide)
+    )
+    (pin "1")
+  )
   (symbol (lib_id "power:GND") (at 172.72 133.35 0) (unit 1)
     (in_bom yes) (on_board yes)
@@
     )
     (property "Datasheet" "" (id 3) (at 214.63 100.33 0)
-      (effects (font (size 1.27 1.27)) hide)
-    )
-    (pin "1")
-  )
-  (symbol (lib_id "power:GND") (at 217.17 69.85 0) (unit 1)
-    (in_bom yes) (on_board yes) (fields_autoplaced)
-    (property "Reference" "#PWR08" (id 0) (at 217.17 76.2 0)
-      (effects (font (size 1.27 1.27)) hide)
-    )
-    (property "Value" "GND" (id 1) (at 217.17 74.93 0))
-    (property "Footprint" "" (id 2) (at 217.17 69.85 0)
-      (effects (font (size 1.27 1.27)) hide)
-    )
-    (property "Datasheet" "" (id 3) (at 217.17 69.85 0)
       (effects (font (size 1.27 1.27)) hide)
     )
@@
     (pin "2")
   )
+  (symbol (lib_id "Device:R_Small") (at 154.94 43.18 90) (unit 1)
+    (in_bom yes) (on_board yes) (fields_autoplaced)
+    (property "Reference" "R?" (id 0) (at 154.94 38.1 90))
+    (property "Value" "1k" (id 1) (at 154.94 40.64 90))
+    (property "Footprint" "" (id 2) (at 154.94 43.18 0)
+      (effects (font (size 1.27 1.27)) hide)
+    )
+    (property "Datasheet" "~" (id 3) (at 154.94 43.18 0)
+      (effects (font (size 1.27 1.27)) hide)
+    )
+    (pin "1")
+    (pin "2")
+  )
+  (symbol (lib_id "Device:R_Small") (at 166.37 31.75 180) (unit 1)
+    (in_bom yes) (on_board yes) (fields_autoplaced)
+    (property "Reference" "R?" (id 0) (at 168.91 31.1149 0)
+      (effects (font (size 1.27 1.27)) (justify right))
+    )
+    (property "Value" "1k" (id 1) (at 168.91 33.6549 0)
+      (effects (font (size 1.27 1.27)) (justify right))
+    )
+    (property "Footprint" "" (id 2) (at 166.37 31.75 0)
+      (effects (font (size 1.27 1.27)) hide)
+    )
+    (property "Datasheet" "~" (id 3) (at 166.37 31.75 0)
+      (effects (font (size 1.27 1.27)) hide)
+    )
+    (pin "1")
+    (pin "2")
+  )
   (symbol (lib_id "Amplifier_Operational:TL074") (at 77.47 163.83 0) (mirror y) (unit 5)
     (in_bom yes) (on_board yes)
@@
     (pin "2")
   )
-  (symbol (lib_id "thonkiconn:AudioJack2_Ground_Switch") (at 212.09 63.5 0) (mirror x) (unit 1)
-    (in_bom yes) (on_board yes)
-    (property "Reference" "J1" (id 0) (at 205.74 63.4999 0)
+  (symbol (lib_id "thonkiconn:AudioJack2_Ground_Switch") (at 142.24 43.18 0) (mirror x) (unit 1)
+    (in_bom yes) (on_board yes)
+    (property "Reference" "J1" (id 0) (at 135.89 43.1799 0)
       (effects (font (size 1.27 1.27)) (justify right))
     )
-    (property "Value" "B_In" (id 1) (at 205.74 66.0399 0)
+    (property "Value" "Gate1_In" (id 1) (at 135.89 45.7199 0)
       (effects (font (size 1.27 1.27)) (justify right))
     )
-    (property "Footprint" "" (id 2) (at 212.09 63.5 0)
-      (effects (font (size 1.27 1.27)) hide)
-    )
-    (property "Datasheet" "~" (id 3) (at 212.09 63.5 0)
+    (property "Footprint" "" (id 2) (at 142.24 43.18 0)
+      (effects (font (size 1.27 1.27)) hide)
+    )
+    (property "Datasheet" "~" (id 3) (at 142.24 43.18 0)
       (effects (font (size 1.27 1.27)) hide)
     )
@@
     (property "Datasheet" "~" (id 3) (at 222.25 95.25 0)
       (effects (font (size 1.27 1.27)) hide)
+    )
+    (pin "1")
+    (pin "2")
+    (pin "3")
+  )
+  (symbol (lib_id "Transistor_BJT:2N3904") (at 163.83 43.18 0) (unit 1)
+    (in_bom yes) (on_board yes) (fields_autoplaced)
+    (property "Reference" "Q?" (id 0) (at 168.91 42.5449 0)
+      (effects (font (size 1.27 1.27)) (justify left))
+    )
+    (property "Value" "2N3904" (id 1) (at 168.91 45.0849 0)
+      (effects (font (size 1.27 1.27)) (justify left))
+    )
+    (property "Footprint" "Package_TO_SOT_THT:TO-92_Inline" (id 2) (at 168.91 45.085 0)
+      (effects (font (size 1.27 1.27) italic) (justify left) hide)
+    )
+    (property "Datasheet" "https://www.onsemi.com/pub/Collateral/2N3903-D.PDF" (id 3) (at 163.83 43.18 0)
+      (effects (font (size 1.27 1.27)) (justify left) hide)
     )
     (pin "1")
@@
       (reference "#PWR025") (unit 1) (value "GND") (footprint "")
     )
+    (path "/06619252-6038-41b4-9120-ebff82779a3e"
+      (reference "#PWR?") (unit 1) (value "+3.3V") (footprint "")
+    )
     (path "/39c42d20-7a90-461b-9133-d9dd1113e1c7"
       (reference "#PWR?") (unit 1) (value "+3.3VA") (footprint "")
     )
+    (path "/45ff6e39-1deb-46ca-a8f7-a2148e535e3b"
+      (reference "#PWR?") (unit 1) (value "GND") (footprint "")
+    )
     (path "/a672c627-9f61-4338-b23e-a341541d50d8"
       (reference "#PWR?") (unit 1) (value "+3.3V") (footprint "")
@@
     )
     (path "/1cace749-dea1-4e12-b191-70f93bf23503"
-      (reference "J1") (unit 1) (value "B_In") (footprint "")
+      (reference "J1") (unit 1) (value "Gate1_In") (footprint "")
     )
     (path "/0436088d-759c-4ef7-a876-ddc66def2f25"
@@
       (reference "L?") (unit 1) (value "L_Small") (footprint "")
     )
+    (path "/d2c178c5-5cea-437c-8c9c-72e0f5c423b0"
+      (reference "Q?") (unit 1) (value "2N3904") (footprint "Package_TO_SOT_THT:TO-92_Inline")
+    )
+    (path "/437e3cd7-018a-4551-a285-0c4021301d2f"
+      (reference "R?") (unit 1) (value "1k") (footprint "")
+    )
     (path "/afdaa434-701d-4d23-a31e-7aa11c74bc7f"
       (reference "R?") (unit 1) (value "100k") (footprint "")
     )
+    (path "/df1e8d51-9668-4e6f-9ba3-89714d0e58e4"
+      (reference "R?") (unit 1) (value "1k") (footprint "")
+    )
     (path "/b534da72-abbc-4d7e-872d-c8cda0f84134"
